File: PCB/KiCAD/CAN_Dashboard_PCB/CAN_Dashboard_PCB.kicad_sch (KiCad schematic)
At the start: 0 parts

Commit message: new
Parts:
- added J1: SN65 Module, symbol Connector_Generic:Conn_01x06
- added J2: OLED, symbol Connector_Generic:Conn_01x04
- added J3: ESP32 Left, symbol Connector_Generic:Conn_01x15
- added J4: ESP32 Right, symbol Connector_Generic:Conn_01x15
Connections:
- new net 3.3V: J1.1 (Pin_1), J4.15 (Pin_15)
- new net CANH: J1.5 (Pin_5)
- new net CANL: J1.6 (Pin_6)
- new net CAN_RX: J1.4 (Pin_4), J4.8 (Pin_8)
- new net CAN_TX: J1.3 (Pin_3), J4.7 (Pin_7)
- new net GND: J1.2 (Pin_2), J4.14 (Pin_14)
- new net GPIO21: J4.5 (Pin_5)
- new net GPIO22: J4.2 (Pin_2)
- new net VIN_5v: J3.15 (Pin_15)
