File: PCB/KiCAD/CAN_Dashboard_PCB/CAN_Dashboard_PCB.kicad_pcb (KiCad board)
At the start: 2 copper layers, 102 x 86.5 mm, 19 parts, among them J1 SN65 Module, J2 OLED, J5 CANH/CANL, J6 Conn_01x02, J7 Conn_01x02, J8 Conn_01x04

Commit message: finished product
Parts:
- J5: value CANH/CANL -> Conn_01x03; footprint TerminalBlock_Phoenix:TerminalBlock_Phoenix_MKDS-1,5-2-5.08_1x02_P5.08mm_Horizontal -> TerminalBlock_Phoenix:TerminalBlock_Phoenix_MKDS-1,5-3-5.08_1x03_P5.08mm_Horizontal
- moved J2 13.0 mm to (159.9, 56.0)
- moved J1 11.7 mm to (146.5, 76.5)
- moved J5 7.62 mm to (167.0, 92.7), turned to 90 degrees
Routing:
- net GND: track 270.1 -> 331.9 mm, vias 1 -> 3
- net /OLED_SCL: track 36.3 -> 54.7 mm, vias 0 -> 1
- net /OLED_SDA: track 27.6 -> 45.8 mm, vias 0 -> 1
- net /CAN_TX: track 59.6 -> 68.0 mm
- net /CAN_RX: track 59.8 -> 51.4 mm, vias 1 -> 2
- net /3V3: track 127.1 -> 132.8 mm, vias 0 -> 1
- net /CANL: track 156.6 -> 158.5 mm, vias 0 -> 1
- net /CANH: track 88.0 -> 86.3 mm, vias 1 -> 2
Other:
- board text added: "+"
- board text added: "120R TERM"
- board text added: "3V3"
- board text added: "5V"
- board text added: "5V BUCK"
- board text added: "9V IN"
- board text added: "CAN Connector"
- board text added: "CAN Module"
- board text added: "CANH"
- board text added: "CANL"
- board text added: "CAN_RX"
- board text added: "CAN_TX"
- board text added: "GND"
- board text added: "IN+"
- board text added: "IN-"
- board text added: "OUT+"
- board text added: "OUT-"
- board text added: "Power Input"
- board text added: "RX"
- board text added: "SCL"
- board text added: "SDA"
- board text added: "TX"
